File: PCB/UART_LCD_MkI.kicad_pcb (KiCad board)
At the start: 2 copper layers, 7 parts, among them U1 CH32V003

Commit message: Updated PCB
Parts:
- added C3: 1uF, Capacitor_SMD:C_0805_2012Metric, F.Cu at (-0.49, 35.0)
- added J1: CONN_DATA, Connector_PinHeader_2.54mm:PinHeader_1x02_P2.54mm_Vertical, F.Cu at (-8.33, 28.6)
- added J2: CONN_POWER, Connector_PinHeader_2.54mm:PinHeader_1x02_P2.54mm_Vertical, F.Cu at (-3.68, 28.6)
- added Q2: AO3400A, Package_TO_SOT_SMD:SOT-23, F.Cu at (-8.21, 35.9)
- added Q3: AO3400A, Package_TO_SOT_SMD:SOT-23, F.Cu at (-8.21, 40.5)
- added R2: 47K, Resistor_SMD:R_0805_2012Metric, F.Cu at (-0.51, 38.0)
- added TP1: VIN, TestPoint:TestPoint_Pad_D1.0mm, F.Cu at (-4.24, 35.0)
- added TP2: GND, TestPoint:TestPoint_Pad_D1.0mm, F.Cu at (-4.24, 38.1)
- added TP3: SWIO, TestPoint:TestPoint_Pad_D1.0mm, F.Cu at (-4.24, 41.1)
- RV1: footprint Resistor_SMD:R_0805_2012Metric -> Potentiometer_THT:Potentiometer_Bourns_3339P_Vertical
- moved RV1 45.4 mm to (56.5, 94.9), turned to -90 degrees
Connections:
- DS1 pad 16: unconnected-(DS1-LED(-)-Pad16) -> Net-(DS1-LED(-))
- U1 pad 10: /LCD_RS -> unconnected-(U1-PC0-Pad10)
- U1 pad 11: /LCD_RW -> /LCD_RS
- U1 pad 12: /LCD_EN -> /LCD_RW
- U1 pad 13: /LCD_DA_0 -> /LCD_EN
- U1 pad 14: /LCD_DA_1 -> /LCD_DA_0
- U1 pad 15: /LCD_DA_2 -> /LCD_DA_1
- U1 pad 16: /LCD_DA_3 -> /LCD_DA_2
- U1 pad 17: unconnected-(U1-PC7-Pad17) -> /LCD_DA_3
- U1 pad 5: unconnected-(U1-PA1-Pad5) -> /BAUD_SEL0
- U1 pad 6: unconnected-(U1-PA2-Pad6) -> /BAUD_SEL1

Commit message: PCB Progress
Parts:
- removed Q3: AO3400A, Package_TO_SOT_SMD:SOT-23
- added JP2: JMP_BL_GND, Jumper:SolderJumper-2_P1.3mm_Open_RoundedPad1.0x1.5mm, B.Cu at (63.6, 26.1)
- added Q1: AO3400A, Package_TO_SOT_SMD:SOT-23, F.Cu at (29.1, 30.3)
- added SW1: BAUD_SEL, Button_Switch_THT:SW_DIP_SPSTx02_Slide_9.78x7.26mm_W7.62mm_P2.54mm, F.Cu at (83.0, 38.9)
- DS1: footprint Display:WC1602A -> Connector_PinHeader_2.54mm:PinHeader_1x16_P2.54mm_Vertical
- J1: value CONN_DATA -> CONN_POWER
- J2: value CONN_POWER -> CONN_DATA
- R2: value 47K -> 4K7
- RV1: value 20K -> 100K; moved to B.Cu
- moved Q2 72.1 mm to (63.3, 26.5)
- moved RV1 66.2 mm to (37.6, 31.4)
- moved TP1 58.8 mm to (54.4, 39.0)
- moved TP2 58.8 mm to (54.4, 41.5)
- moved TP3 58.8 mm to (54.4, 44.0)
- moved C1 53.8 mm to (32.3, 34.1), turned to -90 degrees
- moved D1 50.8 mm to (35.1, 34.1), turned to -90 degrees
- moved JP1 49.1 mm to (35.1, 36.9), turned to 0 degrees
- moved C2 48.3 mm to (37.9, 34.1), turned to -90 degrees
- moved C3 42.2 mm to (41.4, 30.1), turned to 180 degrees
- moved J1 33.7 mm to (25.4, 27.9)
- moved U1 32.5 mm to (43.1, 35.1), turned to -90 degrees
- moved R2 31.5 mm to (29.0, 27.1)
- moved J2 29.9 mm to (25.4, 35.6)
- moved DS1 5.66 mm to (25.4, 22.9), turned to 90 degrees
Connections:
- J1 pad 1: /UART_IN -> /VBUS_VIN
- J1 pad 2: GND -> /VBUS_GND
- J2 pad 1: /VBUS_VIN -> /UART_RX
Routing:
- net /VBUS_VIN: track 0.00 -> 29.0 mm, vias 0 -> 1
- net /LCD_CONTRAST: track 0.00 -> 7.91 mm
- net Net-(D1-A): track 0.00 -> 7.58 mm, vias 0 -> 1
- net GND: track 0.00 -> 6.24 mm, vias 0 -> 7
- net Net-(DS1-LED(-)): track 0.00 -> 5.23 mm, vias 0 -> 1
- net /VBUS_GND: track 0.00 -> 4.63 mm
- net Net-(D1-COM): track 0.00 -> 2.81 mm
- net /LCD_RS: track 0.00 -> 2.39 mm, vias 0 -> 1
- net Net-(Q1-G): track 0.00 -> 2.33 mm
- net /LCD_EN: track 0.00 -> 1.39 mm, vias 0 -> 1
- net /LCD_DA_3: track 0.00 -> 1.39 mm, vias 0 -> 1
- net /LCD_DA_1: track 0.00 -> 1.39 mm, vias 0 -> 1
- net /LCD_RW: track 0.00 -> 1.04 mm, vias 0 -> 1
- net /LCD_DA_2: track 0.00 -> 1.04 mm, vias 0 -> 1
- net /LCD_DA_0: track 0.00 -> 1.04 mm, vias 0 -> 1
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