File: PCB/003-UART-1602.kicad_sch (KiCad schematic)
At the start: 18 parts, among them J1 CONN_POWER, J2 CONN_DATA, Q1 AO3400A, Q2 AO3400A, SW1 BAUD_SEL, U1 CH32V003

Commit message: Changed Project Name
Other:
- title: UART_LCD -> 003-UART-1602
Changed lines of the file:
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@@
 	(paper "A4")
 	(title_block
-		(title "UART_LCD")
-		(date "2024-12-15")
+		(title "003-UART-1602")
+		(date "2024-12-16")
 		(rev "MkI")
 		(company "ADBeta")

Commit message: Added DIP Switch to PCB
Parts:
- SW1: footprint Button_Switch_THT:SW_DIP_SPSTx02_Slide_9.78x7.26mm_W7.62mm_P2.54mm -> Button_Switch_SMD:SW_DIP_SPSTx02_Slide_Copal_CHS-02B_W7.62mm_P1.27mm
Changed lines of the file:
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@@
 			)
 		)
-		(property "Footprint" "Button_Switch_THT:SW_DIP_SPSTx02_Slide_9.78x7.26mm_W7.62mm_P2.54mm"
+		(property "Footprint" "Button_Switch_SMD:SW_DIP_SPSTx02_Slide_Copal_CHS-02B_W7.62mm_P1.27mm"
 			(at 38.735 57.15 0)
 			(effects

Commit message: Almost Final PCB
Parts:
- JP1: value JMP_V0_GND -> JMP_V0
- JP2: value JMP_BL_GND -> JMP_BL
Changed lines of the file:
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@@
 			)
 		)
-		(property "Value" "JMP_V0_GND"
+		(property "Value" "JMP_V0"
 			(at 259.08 33.02 0)
 			(effects
@@
 			)
 		)
-		(property "Value" "JMP_BL_GND"
+		(property "Value" "JMP_BL"
 			(at 193.04 85.09 0)
 			(effects
