File: PCB/003-UART-1602.kicad_sch (KiCad schematic)
At the start: 18 parts, among them J1 CONN_POWER, J2 CONN_DATA, Q1 AO3400A, Q2 AO3400A, SW1 BAUD_SEL, U1 CH32V003

Commit message: MkII PCB Design started
Parts:
- removed J1: CONN_POWER, Connector_PinHeader_2.54mm:PinHeader_1x02_P2.54mm_Vertical, symbol Connector:Conn_01x02_Pin
- removed J2: CONN_DATA, Connector_PinHeader_2.54mm:PinHeader_1x02_P2.54mm_Vertical, symbol Connector:Conn_01x02_Pin
- removed Q1: AO3400A, Package_TO_SOT_SMD:SOT-23, symbol Transistor_FET:AO3400A
- added J1: CONN_INPUT, Connector_PinHeader_2.54mm:PinHeader_1x04_P2.54mm_Vertical, symbol Connector:Conn_01x04_Pin
- added Q1: AO3401A, Package_TO_SOT_SMD:SOT-23, symbol Transistor_FET:AO3401A
- R2: renamed from RV1; footprint Potentiometer_THT:Potentiometer_Bourns_3339P_Vertical -> Potentiometer_THT:Potentiometer_Piher_PT-6-V_Vertical
- renumbered R2 to R1
Connections:
- net GND: now also R1.1, J1.2 (Pin_2), J1.4 (Pin_4)
- net UART_RX: now also J1.3 (Pin_3)
- net VBUS_VIN: now also R2.1, Q1.2 (S); no longer R1.1, R2.3
- net at C2.1, D1.1 (A), JP1.2 (B): now also R2.3; no longer R2.1
- net at R1.2: now also Q1.1 (G)
- new net VIN_HOT: J1.1 (Pin_1), Q1.3 (D)
Other:
- moved on the sheet: C3, DS1, JP2, Q2, R1, R2, SW1, TP1, TP2, TP3, U1
