File: PCB/003-UART-1602.kicad_pcb (KiCad board)
At the start: 2 copper layers, 42 x 20 mm, 18 parts, among them J1 CONN_POWER, J2 CONN_DATA, Q1 AO3400A, Q2 AO3400A, SW1 BAUD_SEL, U1 CH32V003

Commit message: MkII PCB Design started
Parts:
- removed J2: CONN_DATA, Connector_PinHeader_2.54mm:PinHeader_1x02_P2.54mm_Vertical
- removed RV1: 100K, Potentiometer_THT:Potentiometer_Bourns_3339P_Vertical
- added R1: 4K7, Resistor_SMD:R_0805_2012Metric, F.Cu at (36.2, 76.1)
- J1: value CONN_POWER -> CONN_INPUT; footprint Connector_PinHeader_2.54mm:PinHeader_1x02_P2.54mm_Vertical -> Connector_PinHeader_2.54mm:PinHeader_1x04_P2.54mm_Vertical
- Q1: value AO3400A -> AO3401A
- R2: value 4K7 -> 100K; footprint Resistor_SMD:R_0805_2012Metric -> Potentiometer_THT:Potentiometer_Piher_PT-6-V_Vertical; moved to B.Cu
- moved R2 6.59 mm to (40.6, 75.0), turned to 90 degrees
- moved Q2 2.57 mm to (69.0, 72.1)
- moved J1 2.18 mm to (32.4, 73.3)
- moved C1 1.40 mm to (40.3, 78.2)
- moved C2 1.40 mm to (45.9, 78.2)
- moved D1 1.40 mm to (43.1, 78.2)
- moved JP1 1.35 mm to (43.1, 79.2)
- moved C3 1.10 mm to (49.5, 73.3)
- moved U1 1.10 mm to (51.1, 78.3)
- moved JP2 0.96 mm to (68.6, 69.3)
- moved TP1 0.91 mm to (55.9, 75.7)
- moved TP2 0.91 mm to (55.9, 78.2)
- moved TP3 0.91 mm to (55.9, 80.8)
- moved Q1 0.40 mm to (36.4, 73.3), turned to 180 degrees
- moved SW1 0.32 mm to (69.0, 78.5)
Connections:
- J1 pad 1: /VBUS_VIN -> /VIN_HOT
- J1 pad 2: /VBUS_GND -> GND
- Q1 pad 2: GND -> /VBUS_VIN
- Q1 pad 3: /VBUS_GND -> /VIN_HOT
- R2 pad 2: Net-(Q1-G) -> /LCD_CONTRAST
Routing:
- net /VBUS_VIN: track 91.6 -> 58.6 mm, vias 2 -> 1
- net /LCD_DA_3: track 25.5 -> 0.99 mm
- net /LCD_DA_2: track 23.7 -> 1.39 mm
- net /LCD_DA_1: track 22.0 -> 0.99 mm
- net /LCD_DA_0: track 20.2 -> 1.39 mm
- net /LCD_RS: track 18.6 -> 0.99 mm
- net /CHRGPMP: track 21.2 -> 4.18 mm, vias 2 -> 0
- net /UART_RX: track 21.4 -> 5.22 mm
- net /LCD_RW: track 17.1 -> 1.39 mm
- net /LCD_EN: track 16.1 -> 0.99 mm
- net /VBUS_GND: track 4.63 -> 0.00 mm
- net Net-(DS1-LED(-)): track 6.73 -> 10.4 mm, vias 1 -> 0
- net /VIN_HOT: track 0.00 -> 3.05 mm
- net /LCD_BL: track 24.8 -> 22.0 mm
- net /BAUD_SEL1: track 22.9 -> 22.2 mm
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